File: Schematics/NL-USBMach2.0/NL-USBMach2.0.kicad_sch (KiCad schematic)
At the start: 12 parts, among them J1 SWD, U1 STM32F103CBTx, U10 LTV-357T, U12 AMS1117-3.3, U2 74HC245, U3 74HC245, U4 LTV-357T, U5 LTV-357T, U6 LTV-357T, U7 LTV-357T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

Commit message: Routed some headers
Parts:
- added J2, J3, J4, J5, J6: Conn_01x04, symbol Connector_Generic:Conn_01x04
- added J7-11: Conn_01x15, symbol Connector_Generic:Conn_01x15
Connections:
- net GND: now also U2.1 (A->B), U2.10 (GND), U2.19 (CE), U3.1 (A->B), U3.10 (GND), U3.19 (CE), J7-11.5 (Pin_5)
- net at U3.2 (A0): now also J6.3 (Pin_3), J7-11.15 (Pin_15)
- net +5V: now reaches U3.20 (VCC)
- net +5V: now also U2.20 (VCC), J2.4 (Pin_4), J3.4 (Pin_4), J4.4 (Pin_4), J5.4 (Pin_4), J6.4 (Pin_4), J7-11.6 (Pin_6), J7-11.7 (Pin_7)
- net at U3.3 (A1): now also J6.2 (Pin_2), J7-11.14 (Pin_14)
- net at U3.4 (A2): now also J5.3 (Pin_3), J7-11.13 (Pin_13)
- net at U3.5 (A3): now also J5.2 (Pin_2), J7-11.12 (Pin_12)
- net at U3.6 (A4): now also J4.3 (Pin_3), J7-11.11 (Pin_11)
- net at U3.7 (A5): now also J4.2 (Pin_2), J7-11.10 (Pin_10)
- net at U3.8 (A6): now also J3.3 (Pin_3), J7-11.9 (Pin_9)
- net at U3.9 (A7): now also J3.2 (Pin_2), J7-11.8 (Pin_8)
- net at U2.2 (A0): now also J5.1 (Pin_1), J6.1 (Pin_1)
- net at U2.3 (A1): now also J2.3 (Pin_3)
- net at U2.4 (A2): now also J2.2 (Pin_2)
- net at U2.5 (A3): now also J7-11.4 (Pin_4)
- net at U2.6 (A4): now also J7-11.3 (Pin_3)
- net at U2.7 (A5): now also J2.1 (Pin_1), J3.1 (Pin_1), J4.1 (Pin_1)
- net at U2.8 (A6): now also J7-11.1 (Pin_1)
- net at U2.9 (A7): now also J7-11.2 (Pin_2)
- net SWDCLK renamed SWCLK
